File: kicad/coruja.kicad_sch (KiCad schematic)
At the start: 21 parts, among them J1 NEO-M8N (GY-GPSV3), J2 Leitor microSD (9 pinos), J3 Display 2,4" 240x320 ST7789V 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, J4 Encoder KY-040, J5 Conversor step-down 12V->5V (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, J6 RGB 10mm anodo comum, J7 BZ1 SFM-27 (fios diretos), J8 Entrada 12V (pos-chave), Q1 BC337 (nao BC547), U1 Raspberry Pi Pico 2 W

Commit message: feat: placa de 120x120 posicionada, roteada e verificada
Fecha o projeto da PCB: contorno, posicionamento, redes e roteamento manual,
com 0 itens desconectados e 0 divergências contra o esquemático.

Medidas (medidas.py)
--------------------
Todos os módulos medidos na peça física, não em catálogo. O conversor e o GPS
a paquímetro; o leitor microSD a partir do arquivo EAGLE que a Adafruit publica
(CC-BY-SA, Limor Fried/Ladyada), conferido contra a peça. Cada número registra
de que ponto a medida foi tomada — foi a ausência dessa informação que tornou
duas leituras irreprodutíveis e custou duas idas e vindas.

Três footprints próprios, porque o KiCad traz footprint de componente e esses
são placas de breakout genéricas, sem padrão de fabricante. O do GPS marca o
U.FL na camada de fabricação: o rabicho tem 8 cm e quem posicionar o módulo
precisa saber por onde o cabo sai.

Posicionamento (planta.py, arranjo.py, ocupacao.py)
---------------------------------------------------
A planta decide onde ficam os cinco módulos, que é onde está a engenharia:
antena longe do conversor chaveado, cartão e USB faceados na traseira, área
proibida sob a antena. O resto é empacotamento, e empacotamento é trabalho de
programa — o colocador varre posições livres contra a área real de cada
footprint.

A placa cresceu de 100x100 para 120x120 depois de medir o aperto: a 100x100 a
ocupação era de 64% e a folga máxima entre peças pequenas ficava em 1,6 mm.
Em 120x120 cai para 44%.

Defeitos que as ferramentas pegaram, e que eu não teria pegado
---------------------------------------------------------------
- zona dentro de footprint é gravada em coordenada ABSOLUTA, ao contrário dos
  pads; a área de restrição da antena do Pico W aterrissou na origem da placa
- a área de ocupação de um footprint circular estava sendo medida por
  amostragem de pontos, e media menor do que é
- nome de rede na placa sem a barra do caminho da folha (104 avisos de paridade)
- Value com o nome do footprint onde d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
Parts:
- J1: value NEO-M8N (GY-GPSV3) -> NEO-M8N (GY-GPS6MV2); footprint Connector_PinHeader_2.54mm:PinHeader_1x04_P2.54mm_Vertical -> coruja:GPS_GY_GPS6MV2
- J2: footprint Connector_PinHeader_2.54mm:PinHeader_1x09_P2.54mm_Vertical -> coruja:Leitor_microSD_Adafruit4682
- J5: footprint Connector_PinHeader_2.54mm:PinHeader_1x04_P2.54mm_Vertical -> coruja:Conversor_LM2596
